File: upl-keyboard.sch (KiCad schematic (older format))
At the start: 33 parts, among them U1 ProMicro

Commit message: update schematic
Parts:
- U1: footprint Keebio-Parts:ArduinoProMicro -> Keebio-Parts:ArduinoProMicro-BackSide
Changed lines of the file:
@@
 F 0 "U1" H 6000 2787 60  0000 C CNN
 F 1 "ProMicro" H 6000 2681 60  0000 C CNN
-F 2 "Keebio-Parts:ArduinoProMicro" V 7050 -550 60  0001 C CNN
+F 2 "Keebio-Parts:ArduinoProMicro-BackSide" V 7050 -550 60  0001 C CNN
 F 3 "" V 7050 -550 60  0001 C CNN
 	1    6000 1950
